Commit message: Added urdf model for the frame of the wheelchair * Added dae design files for the basic components. * Added urdf models for the basic components. * Added urdf model for the frame of the wheelchair.

File: software/ros/src/pvcchair_description/urdf/old/pvcchair.xacro (robot description, xacro)
@@ -9,7 +9,7 @@
   <xacro:property name="height3" value="1" /> <!-- Link 3 -->
   <!-- Import all Gazebo-customization elements, including Gazebo colors -->
-  <xacro:include filename="$(find pvcchair_description)/urdf/pvcchair.gazebo" />
+  <xacro:include filename="$(find pvcchair_description)/urdf/old/pvcchair.gazebo" />
   <!-- Import Rviz colors -->
-  <xacro:include filename="$(find pvcchair_description)/urdf/materials.xacro" />
+  <xacro:include filename="$(find pvcchair_description)/urdf/old/materials.xacro" />
   <!-- Used for fixing robot to Gazebo 'base_link' -->
   <link name="world" />
@@ -23,5 +23,5 @@
       <origin xyz="0 0 ${height1/2}" rpy="0 0 0"/>
       <geometry>
-	    <box size="${width} ${width} ${height1}"/>
+      <box size="${width} ${width} ${height1}"/>
       </geometry>
     </collision>
@@ -29,5 +29,5 @@
       <origin xyz="0 0 ${height1/2}" rpy="0 0 0"/>
       <geometry>
-	    <box size="${width} ${width} ${height1}"/>
+      <box size="${width} ${width} ${height1}"/>
       </geometry>
       <material name="orange"/>
@@ -37,7 +37,7 @@
       <mass value="${mass}"/>
       <inertia
-	      ixx="${mass / 12.0 * (width*width + height1*height1)}" ixy="0.0" ixz="0.0"
-	      iyy="${mass / 12.0 * (height1*height1 + width*width)}" iyz="0.0"
-	      izz="${mass / 12.0 * (width*width + width*width)}"/>
+        ixx="${mass / 12.0 * (width*width + height1*height1)}" ixy="0.0" ixz="0.0"
+        iyy="${mass / 12.0 * (height1*height1 + width*width)}" iyz="0.0"
+        izz="${mass / 12.0 * (width*width + width*width)}"/>
     </inertial>
   </link>
