Commit message: Updated urdf models * Fixed mesh names in urdfs to comply with latest xacro requirements. * Refactored urdf parameters and placed them in parameters.urdf.xacro

File: software/ros/src/pvcchair_description/urdf/connectors/ca.urdf.xacro (robot description, xacro)
@@ -1,5 +1,5 @@
 <?xml version="1.0"?>
 <robot name="ca-4-way-t-connect" xmlns:xacro="http://www.ros.org/wiki/xacro">
-  <xacro:property name="ca-mesh">
+  <xacro:property name="ca_mesh">
     <mesh filename="package://pvcchair_description/meshes/connectors/ca_4_way_t_connect.dae" />
   </xacro:property>
@@ -16,5 +16,5 @@
         <origin xyz="0 0 0" rpy="0 0 ${-pi/2}" />
         <geometry>
-          <xacro:insert_block name="ca-mesh" />
+          <xacro:insert_block name="ca_mesh" />
         </geometry>
       </visual>
@@ -22,5 +22,5 @@
         <origin xyz="0 0 0" rpy="0 0 ${-pi/2}" />
         <geometry>
-          <xacro:insert_block name="ca-mesh" />
+          <xacro:insert_block name="ca_mesh" />
         </geometry>
       </collision>

File: software/ros/src/pvcchair_description/urdf/connectors/cb.urdf.xacro (robot description, xacro)
@@ -1,5 +1,5 @@
 <?xml version="1.0"?>
 <robot name="cb" xmlns:xacro="http://www.ros.org/wiki/xacro">
-  <xacro:property name="cb-mesh">
+  <xacro:property name="cb_mesh">
     <mesh filename="package://pvcchair_description/meshes/connectors/cb_5_way_t_connect.dae" />
   </xacro:property>
@@ -16,5 +16,5 @@
         <origin xyz="0 0 0" rpy="0 0 ${-pi/2}" />
         <geometry>
-          <xacro:insert_block name="cb-mesh" />
+          <xacro:insert_block name="cb_mesh" />
         </geometry>
       </visual>
@@ -22,5 +22,5 @@
         <origin xyz="0 0 0" rpy="0 0 ${-pi/2}" />
         <geometry>
-          <xacro:insert_block name="cb-mesh" />
+          <xacro:insert_block name="cb_mesh" />
         </geometry>
       </collision>

File: software/ros/src/pvcchair_description/urdf/connectors/cc.urdf.xacro (robot description, xacro)
@@ -1,5 +1,5 @@
 <?xml version="1.0"?>
 <robot name="cc" xmlns:xacro="http://www.ros.org/wiki/xacro">
-  <xacro:property name="cc-mesh">
+  <xacro:property name="cc_mesh">
     <mesh filename="package://pvcchair_description/meshes/connectors/cc_3_way_y_connect.dae" />
   </xacro:property>
@@ -16,5 +16,5 @@
         <origin xyz="0 0 0" rpy="0 0 ${pi/2}" />
         <geometry>
-          <xacro:insert_block name="cc-mesh" />
+          <xacro:insert_block name="cc_mesh" />
         </geometry>
       </visual>
@@ -22,5 +22,5 @@
         <origin xyz="0 0 0" rpy="0 0 ${pi/2}" />
         <geometry>
-          <xacro:insert_block name="cc-mesh" />
+          <xacro:insert_block name="cc_mesh" />
         </geometry>
       </collision>

File: software/ros/src/pvcchair_description/urdf/connectors/cd.urdf.xacro (robot description, xacro)
@@ -1,5 +1,5 @@
 <?xml version="1.0"?>
 <robot name="cd" xmlns:xacro="http://www.ros.org/wiki/xacro">
-  <xacro:property name="cd-mesh">
+  <xacro:property name="cd_mesh">
     <mesh filename="package://pvcchair_description/meshes/connectors/cd_2_way_elbow.dae" />
   </xacro:property>
@@ -16,5 +16,5 @@
         <origin xyz="0 0 0" rpy="0 0 ${pi/2}" />
         <geometry>
-          <xacro:insert_block name="cd-mesh" />
+          <xacro:insert_block name="cd_mesh" />
         </geometry>
       </visual>
@@ -22,5 +22,5 @@
         <origin xyz="0 0 0" rpy="0 0 ${pi/2}" />
         <geometry>
-          <xacro:insert_block name="cd-mesh" />
+          <xacro:insert_block name="cd_mesh" />
         </geometry>
       </collision>

File: software/ros/src/pvcchair_description/urdf/connectors/ce.urdf.xacro (robot description, xacro)
@@ -1,5 +1,5 @@
 <?xml version="1.0"?>
 <robot name="ce" xmlns:xacro="http://www.ros.org/wiki/xacro">
-  <xacro:property name="ce-mesh">
+  <xacro:property name="ce_mesh">
     <mesh filename="package://pvcchair_description/meshes/connectors/ce_3_way_t_connect.dae" />
   </xacro:property>
@@ -16,5 +16,5 @@
         <origin xyz="0 0 0" rpy="0 0 ${-pi/2}" />
         <geometry>
-          <xacro:insert_block name="ce-mesh" />
+          <xacro:insert_block name="ce_mesh" />
         </geometry>
       </visual>
@@ -22,5 +22,5 @@
         <origin xyz="0 0 0" rpy="0 0 ${-pi/2}" />
         <geometry>
-          <xacro:insert_block name="ce-mesh" />
+          <xacro:insert_block name="ce_mesh" />
         </geometry>
       </collision>

File: software/ros/src/pvcchair_description/urdf/connectors/cf.urdf.xacro (robot description, xacro)
@@ -1,5 +1,5 @@
 <?xml version="1.0"?>
 <robot name="cf" xmlns:xacro="http://www.ros.org/wiki/xacro">
-  <xacro:property name="cf-mesh">
+  <xacro:property name="cf_mesh">
     <mesh filename="package://pvcchair_description/meshes/connectors/cf_3_way_slip.dae" />
   </xacro:property>
@@ -16,5 +16,5 @@
         <origin xyz="0 0 0" rpy="0 0 ${-pi/2}" />
         <geometry>
-          <xacro:insert_block name="cf-mesh" />
+          <xacro:insert_block name="cf_mesh" />
         </geometry>
       </visual>
@@ -22,5 +22,5 @@
         <origin xyz="0 0 0" rpy="0 0 ${-pi/2}" />
         <geometry>
-          <xacro:insert_block name="cf-mesh" />
+          <xacro:insert_block name="cf_mesh" />
         </geometry>
       </collision>

File: software/ros/src/pvcchair_description/urdf/connectors/connectors.urdf.xacro (robot description, xacro)
@@ -1,5 +1,4 @@
 <?xml version="1.0"?>
 <robot name="connectors" xmlns:xacro="http://www.ros.org/wiki/xacro">
-  <xacro:property name="c_joint_offset" value="0.0125" />
   <xacro:include filename="$(find pvcchair_description)/urdf/connectors/ca.urdf.xacro" />
   <xacro:include filename="$(find pvcchair_description)/urdf/connectors/cb.urdf.xacro" />

File: software/ros/src/pvcchair_description/urdf/parts.urdf.xacro (robot description, xacro)
@@ -1,8 +1,5 @@
 <?xml version="1.0"?>
 <robot name="parts" xmlns:xacro="http://www.ros.org/wiki/xacro">
-  <xacro:property name="pi" value="3.1415926535897931" />
-  <xacro:property name="back_angle" value="20" />  <!-- in degrees -->
-  <xacro:property name="rest_angle" value="48.8" />  <!-- in degrees -->
-  <xacro:property name="lock_angle" value="20.5" />  <!-- in degrees -->
+  <xacro:include filename="$(find pvcchair_description)/urdf/parameters.urdf.xacro" />
   <xacro:include filename="$(find pvcchair_description)/urdf/piping/piping.urdf.xacro" />
   <xacro:include filename="$(find pvcchair_description)/urdf/connectors/connectors.urdf.xacro" />

File: software/ros/src/pvcchair_description/urdf/piping/p1.urdf.xacro (robot description, xacro)
@@ -1,8 +1,7 @@
 <?xml version="1.0"?>
 <robot name="p1-left-n-right-base" xmlns:xacro="http://www.ros.org/wiki/xacro">
-  <xacro:property name="p1-mesh">
+  <xacro:property name="p1_mesh">
     <mesh filename="package://pvcchair_description/meshes/piping/p1_left_n_right_base.dae" />
   </xacro:property>
-  <xacro:property name="p1_length" value="0.203200" />
   <xacro:macro name="p1" params="suffix">
     <link name="p1_${suffix}">
@@ -17,5 +16,5 @@
         <origin xyz="0 0 0" rpy="0 ${pi/2} 0" />
         <geometry>
-          <xacro:insert_block name="p1-mesh" />
+          <xacro:insert_block name="p1_mesh" />
         </geometry>
       </visual>
@@ -23,5 +22,5 @@
         <origin xyz="0 0 0" rpy="0 ${pi/2} 0" />
         <geometry>
-          <xacro:insert_block name="p1-mesh" />
+          <xacro:insert_block name="p1_mesh" />
         </geometry>
       </collision>

File: software/ros/src/pvcchair_description/urdf/piping/p2.urdf.xacro (robot description, xacro)
@@ -1,8 +1,7 @@
 <?xml version="1.0"?>
 <robot name="p2" xmlns:xacro="http://www.ros.org/wiki/xacro">
-  <xacro:property name="p2-mesh">
+  <xacro:property name="p2_mesh">
     <mesh filename="package://pvcchair_description/meshes/piping/p2_front_n_back_base.dae" />
   </xacro:property>
-  <xacro:property name="p2_length" value="0.241300" />
   <xacro:macro name="p2" params="suffix">
     <link name="p2_${suffix}">
@@ -17,5 +16,5 @@
         <origin xyz="0 0 0" rpy="0 ${pi/2} 0" />
         <geometry>
-          <xacro:insert_block name="p2-mesh" />
+          <xacro:insert_block name="p2_mesh" />
         </geometry>
       </visual>
@@ -23,5 +22,5 @@
         <origin xyz="0 0 0" rpy="0 ${pi/2} 0" />
         <geometry>
-          <xacro:insert_block name="p2-mesh" />
+          <xacro:insert_block name="p2_mesh" />
         </geometry>
       </collision>

File: software/ros/src/pvcchair_description/urdf/piping/p3.urdf.xacro (robot description, xacro)
@@ -1,8 +1,7 @@
 <?xml version="1.0"?>
 <robot name="p3" xmlns:xacro="http://www.ros.org/wiki/xacro">
-  <xacro:property name="p3-mesh">
+  <xacro:property name="p3_mesh">
     <mesh filename="package://pvcchair_description/meshes/piping/p3_left_n_right_back_upright.dae" />
   </xacro:property>
-  <xacro:property name="p3_length" value="0.101600" />
   <xacro:macro name="p3" params="suffix">
     <link name="p3_${suffix}">
@@ -17,5 +16,5 @@
         <origin xyz="0 0 0" rpy="0 ${pi/2} 0" />
         <geometry>
-          <xacro:insert_block name="p3-mesh" />
+          <xacro:insert_block name="p3_mesh" />
         </geometry>
       </visual>
@@ -23,5 +22,5 @@
         <origin xyz="0 0 0" rpy="0 ${pi/2} 0" />
         <geometry>
-          <xacro:insert_block name="p3-mesh" />
+          <xacro:insert_block name="p3_mesh" />
         </geometry>
       </collision>

File: software/ros/src/pvcchair_description/urdf/piping/p4.urdf.xacro (robot description, xacro)
@@ -1,8 +1,7 @@
 <?xml version="1.0"?>
 <robot name="p4" xmlns:xacro="http://www.ros.org/wiki/xacro">
-  <xacro:property name="p4-mesh">
+  <xacro:property name="p4_mesh">
     <mesh filename="package://pvcchair_description/meshes/piping/p4_footrest_base.dae" />
   </xacro:property>
-  <xacro:property name="p4_length" value="0.088900" />
   <xacro:macro name="p4" params="suffix">
     <link name="p4_${suffix}">
@@ -17,5 +16,5 @@
         <origin xyz="0 0 0" rpy="0 ${pi/2} 0" />
         <geometry>
-          <xacro:insert_block name="p4-mesh" />
+          <xacro:insert_block name="p4_mesh" />
         </geometry>
       </visual>
@@ -23,5 +22,5 @@
         <origin xyz="0 0 0" rpy="0 ${pi/2} 0" />
         <geometry>
-          <xacro:insert_block name="p4-mesh" />
+          <xacro:insert_block name="p4_mesh" />
         </geometry>
       </collision>

File: software/ros/src/pvcchair_description/urdf/piping/p5.urdf.xacro (robot description, xacro)
@@ -1,8 +1,7 @@
 <?xml version="1.0"?>
 <robot name="p5" xmlns:xacro="http://www.ros.org/wiki/xacro">
-  <xacro:property name="p5-mesh">
+  <xacro:property name="p5_mesh">
     <mesh filename="package://pvcchair_description/meshes/piping/p5_back_rest_vert.dae" />
   </xacro:property>
-  <xacro:property name="p5_length" value="0.152400" />
   <xacro:macro name="p5" params="suffix">
     <link name="p5_${suffix}">
@@ -17,5 +16,5 @@
         <origin xyz="0 0 0" rpy="0 ${pi/2} 0" />
         <geometry>
-          <xacro:insert_block name="p5-mesh" />
+          <xacro:insert_block name="p5_mesh" />
         </geometry>
       </visual>
@@ -23,5 +22,5 @@
         <origin xyz="0 0 0" rpy="0 ${pi/2} 0" />
         <geometry>
-          <xacro:insert_block name="p5-mesh" />
+          <xacro:insert_block name="p5_mesh" />
         </geometry>
       </collision>

File: software/ros/src/pvcchair_description/urdf/piping/p6.urdf.xacro (robot description, xacro)
@@ -1,8 +1,7 @@
 <?xml version="1.0"?>
 <robot name="p6" xmlns:xacro="http://www.ros.org/wiki/xacro">
-  <xacro:property name="p6-mesh">
+  <xacro:property name="p6_mesh">
     <mesh filename="package://pvcchair_description/meshes/piping/p6_back_rest_horz.dae" />
   </xacro:property>
-  <xacro:property name="p6_length" value="0.146050" />
   <xacro:macro name="p6" params="suffix">
     <link name="p6_${suffix}">
@@ -17,5 +16,5 @@
         <origin xyz="0 0 0" rpy="0 ${pi/2} 0" />
         <geometry>
-          <xacro:insert_block name="p6-mesh" />
+          <xacro:insert_block name="p6_mesh" />
         </geometry>
       </visual>
@@ -23,5 +22,5 @@
         <origin xyz="0 0 0" rpy="0 ${pi/2} 0" />
         <geometry>
-          <xacro:insert_block name="p6-mesh" />
+          <xacro:insert_block name="p6_mesh" />
         </geometry>
       </collision>

File: software/ros/src/pvcchair_description/urdf/piping/p7.urdf.xacro (robot description, xacro)
@@ -1,8 +1,7 @@
 <?xml version="1.0"?>
 <robot name="p7" xmlns:xacro="http://www.ros.org/wiki/xacro">
-  <xacro:property name="p7-mesh">
+  <xacro:property name="p7_mesh">
     <mesh filename="package://pvcchair_description/meshes/piping/p7_adjusting_pipe_horz.dae" />
   </xacro:property>
-  <xacro:property name="p7_length" value="0.285750" />
   <xacro:macro name="p7" params="suffix">
     <link name="p7_${suffix}">
@@ -17,5 +16,5 @@
         <origin xyz="0 0 0" rpy="0 ${pi/2} 0" />
         <geometry>
-          <xacro:insert_block name="p7-mesh" />
+          <xacro:insert_block name="p7_mesh" />
         </geometry>
       </visual>
@@ -23,5 +22,5 @@
         <origin xyz="0 0 0" rpy="0 ${pi/2} 0" />
         <geometry>
-          <xacro:insert_block name="p7-mesh" />
+          <xacro:insert_block name="p7_mesh" />
         </geometry>
       </collision>

File: software/ros/src/pvcchair_description/urdf/piping/p8.urdf.xacro (robot description, xacro)
@@ -1,8 +1,7 @@
 <?xml version="1.0"?>
 <robot name="p8" xmlns:xacro="http://www.ros.org/wiki/xacro">
-  <xacro:property name="p8-mesh">
+  <xacro:property name="p8_mesh">
     <mesh filename="package://pvcchair_description/meshes/piping/p8_arm_rest_hgt_back_n_arms.dae" />
   </xacro:property>
-  <xacro:property name="p8_length" value="0.038100" />
   <xacro:macro name="p8" params="suffix">
     <link name="p8_${suffix}">
@@ -17,5 +16,5 @@
         <origin xyz="0 0 0" rpy="0 ${pi/2} 0" />
         <geometry>
-          <xacro:insert_block name="p8-mesh" />
+          <xacro:insert_block name="p8_mesh" />
         </geometry>
       </visual>
@@ -23,5 +22,5 @@
         <origin xyz="0 0 0" rpy="0 ${pi/2} 0" />
         <geometry>
-          <xacro:insert_block name="p8-mesh" />
+          <xacro:insert_block name="p8_mesh" />
         </geometry>
       </collision>

File: software/ros/src/pvcchair_description/urdf/piping/p9.urdf.xacro (robot description, xacro)
@@ -1,8 +1,7 @@
 <?xml version="1.0"?>
 <robot name="p9" xmlns:xacro="http://www.ros.org/wiki/xacro">
-  <xacro:property name="p9-mesh">
+  <xacro:property name="p9_mesh">
     <mesh filename="package://pvcchair_description/meshes/piping/p9_connects_all.dae" />
   </xacro:property>
-  <xacro:property name="p9_length" value="0.038100" />
   <xacro:macro name="p9" params="suffix">
     <link name="p9_${suffix}">
@@ -17,5 +16,5 @@
         <origin xyz="0 0 0" rpy="0 ${pi/2} 0" />
         <geometry>
-          <xacro:insert_block name="p9-mesh" />
+          <xacro:insert_block name="p9_mesh" />
         </geometry>
       </visual>
@@ -23,5 +22,5 @@
         <origin xyz="0 0 0" rpy="0 ${pi/2} 0" />
         <geometry>
-          <xacro:insert_block name="p9-mesh" />
+          <xacro:insert_block name="p9_mesh" />
         </geometry>
       </collision>
