Commit message: Added urdf models for gearbox plates, wheels and casters

File: software/ros/src/pvcchair_description/urdf/base.urdf.xacro (robot description, xacro)
@@ -4,5 +4,5 @@
   <link name="base_link" />
   <joint name="base_joint" type="fixed">
-    <origin xyz="0 0 0.12" rpy="0 0 0" />
+    <origin xyz="0 0 ${base_level}" rpy="0 0 0" />
     <parent link="base_footprint" />
     <child link="base_link" />
@@ -208,3 +208,60 @@
     <child link="p9_5" />
   </joint>
+  <!-- Gearbox Plates -->
+  <xacro:gearbox_plate suffix="right" />
+  <joint name="gearbox_plate_right_joint" type="fixed">
+    <origin xyz="${-gearbox_plate_offset} -0.015 ${-gearbox_plate_offset}" rpy="0 ${pi} 0" />
+    <parent link="cb_0" />
+    <child link="gearbox_plate_right" />
+  </joint>
+  <xacro:gearbox_plate suffix="left" />
+  <joint name="gearbox_plate_left_joint" type="fixed">
+    <origin xyz="${-gearbox_plate_offset} -0.015 ${gearbox_plate_offset}" rpy="0 0 ${pi}" />
+    <parent link="cb_1" />
+    <child link="gearbox_plate_left" />
+  </joint>
+  <!-- Wheels -->
+  <xacro:wheel suffix="right" />
+  <joint name="wheel_right_joint" type="continuous">
+    <axis xyz="0 0 -1" />
+    <origin xyz="0 -0.02 0" rpy="${pi/2} 0 0" />
+    <parent link="wheel_axle_right" />
+    <child link="wheel_right" />
+  </joint>
+  <xacro:wheel suffix="left" />
+  <joint name="wheel_left_joint" type="continuous">
+    <axis xyz="0 0 -1" />
+    <origin xyz="0 0.02 0" rpy="${pi/2} 0 0" />
+    <parent link="wheel_axle_left" />
+    <child link="wheel_left" />
+  </joint>
+  <!-- Casters -->
+  <link name="swivel_right" />
+  <joint name="swivel_right_joint" type="continuous">
+    <axis xyz="0 0 1" />
+    <origin xyz="0 ${swivel_offset} ${c_joint_offset}" rpy="${pi} 0 ${pi/2}" />
+    <parent link="ca_0" />
+    <child link="swivel_right" />
+  </joint>
+  <link name="swivel_left" />
+  <joint name="swivel_left_joint" type="continuous">
+    <axis xyz="0 0 1" />
+    <origin xyz="0 ${swivel_offset} ${-c_joint_offset}" rpy="0 0 ${pi/2}" />
+    <parent link="ca_1" />
+    <child link="swivel_left" />
+  </joint>
+  <xacro:caster suffix="right" />
+  <joint name="caster_right_joint" type="continuous">
+    <axis xyz="0 0 -1" />
+    <origin xyz="0 0 ${- p9_length - c_joint_offset - base_level + caster_radius}" rpy="${pi/2} 0 0" />
+    <parent link="swivel_right" />
+    <child link="caster_right" />
+  </joint>
+  <xacro:caster suffix="left" />
+  <joint name="caster_left_joint" type="continuous">
+    <axis xyz="0 0 -1" />
+    <origin xyz="0 0 ${- p9_length - c_joint_offset - base_level + caster_radius}" rpy="${pi/2} 0 0" />
+    <parent link="swivel_left" />
+    <child link="caster_left" />
+  </joint>
 </robot>

File: software/ros/src/pvcchair_description/urdf/connectors/ca.urdf.xacro (robot description, xacro)
@@ -1,4 +1,4 @@
 <?xml version="1.0"?>
-<robot name="ca-4-way-t-connect" xmlns:xacro="http://www.ros.org/wiki/xacro">
+<robot name="ca" xmlns:xacro="http://www.ros.org/wiki/xacro">
   <xacro:property name="ca_mesh">
     <mesh filename="package://pvcchair_description/meshes/connectors/ca_4_way_t_connect.dae" />

File: software/ros/src/pvcchair_description/urdf/parameters.urdf.xacro (robot description, xacro)
@@ -12,4 +12,9 @@
   <xacro:property name="p9_length" value="0.038100" />
   <xacro:property name="c_joint_offset" value="0.0125" />
+  <xacro:property name="gearbox_plate_offset" value="0.01" />
+  <xacro:property name="wheel_radius" value="0.0762" />
+  <xacro:property name="caster_radius" value="0.0508" />
+  <xacro:property name="swivel_offset" value="0.02" />
+  <xacro:property name="base_level" value="0.12" />
   <xacro:property name="back_angle" value="20" />  <!-- in degrees -->
   <xacro:property name="rest_angle" value="48.8" />

File: software/ros/src/pvcchair_description/urdf/parts.urdf.xacro (robot description, xacro)
@@ -4,3 +4,4 @@
   <xacro:include filename="$(find pvcchair_description)/urdf/piping/piping.urdf.xacro" />
   <xacro:include filename="$(find pvcchair_description)/urdf/connectors/connectors.urdf.xacro" />
+  <xacro:include filename="$(find pvcchair_description)/urdf/wheels/parts.urdf.xacro" />
 </robot>

File: software/ros/src/pvcchair_description/urdf/piping/p1.urdf.xacro (robot description, xacro)
@@ -1,4 +1,4 @@
 <?xml version="1.0"?>
-<robot name="p1-left-n-right-base" xmlns:xacro="http://www.ros.org/wiki/xacro">
+<robot name="p1" xmlns:xacro="http://www.ros.org/wiki/xacro">
   <xacro:property name="p1_mesh">
     <mesh filename="package://pvcchair_description/meshes/piping/p1_left_n_right_base.dae" />

Commit message: Fixed caster relative positions

File: software/ros/src/pvcchair_description/urdf/base.urdf.xacro (robot description, xacro)
@@ -254,5 +254,5 @@
   <joint name="caster_right_joint" type="continuous">
     <axis xyz="0 0 -1" />
-    <origin xyz="0 0 ${- p9_length - c_joint_offset - base_level + caster_radius}" rpy="${pi/2} 0 0" />
+    <origin xyz="${- caster_radius + 0.005} 0 ${- p9_length - c_joint_offset - base_level + caster_radius}" rpy="${pi/2} 0 0" />
     <parent link="swivel_right" />
     <child link="caster_right" />
@@ -261,5 +261,5 @@
   <joint name="caster_left_joint" type="continuous">
     <axis xyz="0 0 -1" />
-    <origin xyz="0 0 ${- p9_length - c_joint_offset - base_level + caster_radius}" rpy="${pi/2} 0 0" />
+    <origin xyz="${- caster_radius + 0.005} 0 ${- p9_length - c_joint_offset - base_level + caster_radius}" rpy="${pi/2} 0 0" />
     <parent link="swivel_left" />
     <child link="caster_left" />
