Commit message: Refactor and clean up urdf description

File: software/ros/pvcchair_description/urdf/includes/parts/caster.xacro (robot description, xacro)
@@ -1,9 +1,14 @@
 <?xml version="1.0"?>
 <robot name="caster" xmlns:xacro="http://www.ros.org/wiki/xacro">
-  <!-- <xacro:property name="gearbox_plate_mesh">
-    <mesh filename="package://pvcchair_description/meshes/caster.dae" />
-  </xacro:property> -->
-  <xacro:macro name="caster" params="suffix">
-    <link name="caster_${suffix}">
+  <xacro:include filename="$(find pvcchair_description)/urdf/includes/parameters.xacro" />
+  <xacro:macro name="caster" params="suffix parent xyz">
+    <link name="swivel_${suffix}_link" />
+    <joint name="swivel_${suffix}" type="continuous">
+      <axis xyz="0 0 1" />
+      <origin xyz="${xyz}" rpy="0 0 0" />
+      <parent link="${parent}" />
+      <child link="swivel_${suffix}_link" />
+    </joint>
+    <link name="caster_${suffix}_link">
       <inertial>
         <mass value="0.040000" />
@@ -18,6 +23,6 @@
           <cylinder radius="${caster_radius}" length="0.0254" />
         </geometry>
-        <material name="Black">
-          <color rgba="0 0 0 1"/>
+        <material name="black">
+          <color rgba="0 0 0 1" />
         </material>
       </visual>
@@ -29,4 +34,10 @@
       </collision>
     </link>
+    <joint name="caster_${suffix}" type="continuous">
+      <axis xyz="0 1 0" />
+      <origin xyz="${-caster_radius+0.005} 0 ${-c_offset-p9_len-base_level+caster_radius}" rpy="0 0 0" />
+      <parent link="swivel_${suffix}_link" />
+      <child link="caster_${suffix}_link" />
+    </joint>
   </xacro:macro>
 </robot>

File: software/ros/pvcchair_description/urdf/includes/parts/gearbox_plate.xacro (robot description, xacro)
@@ -1,9 +1,6 @@
 <?xml version="1.0"?>
 <robot name="gearbox_plate" xmlns:xacro="http://www.ros.org/wiki/xacro">
-  <xacro:property name="gearbox_plate_mesh">
-    <mesh filename="package://pvcchair_description/meshes/gearbox_plate.dae" />
-  </xacro:property>
-  <xacro:macro name="gearbox_plate" params="suffix">
-    <link name="gearbox_plate_${suffix}">
+  <xacro:macro name="gearbox_plate" params="suffix parent xyz">
+    <link name="gearbox_plate_${suffix}_link">
       <inertial>
         <mass value="0.080099" />
@@ -16,5 +13,5 @@
         <origin xyz="0 0 0" rpy="0 0 0" />
         <geometry>
-          <xacro:insert_block name="gearbox_plate_mesh" />
+          <mesh filename="package://pvcchair_description/meshes/gearbox_plate.dae" />
         </geometry>
       </visual>
@@ -22,13 +19,12 @@
         <origin xyz="0 0 0" rpy="0 0 0" />
         <geometry>
-          <xacro:insert_block name="gearbox_plate_mesh" />
+          <mesh filename="package://pvcchair_description/meshes/gearbox_plate.dae" />
         </geometry>
       </collision>
     </link>
-    <link name="wheel_axle_${suffix}" />
-    <joint name="plate_wheel_${suffix}_joint" type="fixed">
-      <origin xyz="-0.052 0 -0.054" rpy="0 0 0" />
-      <parent link="gearbox_plate_${suffix}" />
-      <child link="wheel_axle_${suffix}" />
+    <joint name="gearbox_plate_${suffix}_joint" type="fixed">
+      <origin xyz="${xyz}" rpy="0 0 0" />
+      <parent link="${parent}" />
+      <child link="gearbox_plate_${suffix}_link" />
     </joint>
   </xacro:macro>

File: software/ros/pvcchair_description/urdf/includes/parts/wheel.xacro (robot description, xacro)
@@ -1,9 +1,7 @@
 <?xml version="1.0"?>
 <robot name="wheel" xmlns:xacro="http://www.ros.org/wiki/xacro">
-  <!-- <xacro:property name="gearbox_plate_mesh">
-    <mesh filename="package://pvcchair_description/meshes/wheel.dae" />
-  </xacro:property> -->
-  <xacro:macro name="wheel" params="suffix">
-    <link name="wheel_${suffix}">
+  <xacro:include filename="$(find pvcchair_description)/urdf/includes/parameters.xacro" />
+  <xacro:macro name="wheel" params="suffix parent xyz">
+    <link name="wheel_${suffix}_link">
       <inertial>
         <mass value="0.020000" />
@@ -18,6 +16,6 @@
           <cylinder radius="${wheel_radius}" length="0.0254" />
         </geometry>
-        <material name="Black">
-          <color rgba="0 0 0 1"/>
+        <material name="black">
+          <color rgba="0 0 0 1" />
         </material>
       </visual>
@@ -29,4 +27,10 @@
       </collision>
     </link>
+    <joint name="wheel_${suffix}" type="continuous">
+      <axis xyz="0 1 0" />
+      <origin xyz="${xyz}" rpy="0 0 0" />
+      <parent link="${parent}" />
+      <child link="wheel_${suffix}_link" />
+    </joint>
   </xacro:macro>
 </robot>

Commit message: Prepare pvcchair for gazebo
* Extend urdf description with the gazebo configuration
* Configure and load controllers in the bringup

File: software/ros/pvcchair_description/urdf/includes/parts/caster.xacro (robot description, xacro)
@@ -3,5 +3,13 @@
   <xacro:include filename="$(find pvcchair_description)/urdf/includes/parameters.xacro" />
   <xacro:macro name="caster" params="suffix parent xyz">
-    <link name="swivel_${suffix}_link" />
+    <link name="swivel_${suffix}_link">
+      <inertial>
+        <mass value="0.2" />
+        <origin xyz="0 0 0" />
+        <inertia ixx="0.000333" ixy="0.000000" ixz="0.000000"
+                                iyy="0.000333" iyz="0.000000"
+                                               izz="0.000333" />
+      </inertial>
+    </link>
     <joint name="swivel_${suffix}" type="continuous">
       <axis xyz="0 0 1" />
