Commit message: Update gazebo extensions for swerve drive base in urdf

File: software/src/pvcchair_description/urdf/includes/parts/swerve_wheel.xacro (robot description, xacro)
@@ -90,5 +90,5 @@
     </link>
     <joint name="${prefix}_caster_r_wheel_joint" type="continuous">
-      <axis xyz="0 1 0" />
+      <axis xyz="0 ${copysign(1,y)} 0" />
       <origin xyz="0 ${box_size/2+wheel_width/2+0.005} 0" rpy="0 0 0" />
       <parent link="${prefix}_caster_rotation_link" />
