Commit message: Parameterize wheel offsets
* Add paremeters that offset the horizontal positioning of the front and rear wheels
* Add parameter that scales the entire model

File: software/src/pvcchair_description/urdf/includes/components/drive.xacro (robot description, xacro)
@@ -8,17 +8,17 @@
       suffix="right"
       parent="${parent}"
-      xyz="${p1_hlen+c_offset-0.042} ${-p2_hlen-c_offset-0.035} ${-base_level+wheel_radius}" />
+      xyz="${p1_hlen+c_offset+front_wheels_offset[0]} ${-p2_hlen-c_offset-front_wheels_offset[1]} ${-base_level+wheel_radius}" />
     <xacro:wheel
       suffix="left"
       parent="${parent}"
-      xyz="${p1_hlen+c_offset-0.042} ${+p2_hlen+c_offset+0.035} ${-base_level+wheel_radius}" />
+      xyz="${p1_hlen+c_offset+front_wheels_offset[0]} ${+p2_hlen+c_offset+front_wheels_offset[1]} ${-base_level+wheel_radius}" />
     <xacro:caster
       suffix="right"
       parent="${parent}"
-      xyz="${-p1_hlen-2*c_offset-p3_len-c_offset+swivel_offset} ${-p2_hlen-c_offset} ${c_offset+p9_len}" />
+      xyz="${-p1_hlen-2*c_offset-p3_len-c_offset+rear_wheels_offset[0]} ${-p2_hlen-c_offset-rear_wheels_offset[1]} ${c_offset+p9_len}" />
     <xacro:caster
       suffix="left"
       parent="${parent}"
-      xyz="${-p1_hlen-2*c_offset-p3_len-c_offset+swivel_offset} ${+p2_hlen+c_offset} ${c_offset+p9_len}" />
+      xyz="${-p1_hlen-2*c_offset-p3_len-c_offset+rear_wheels_offset[0]} ${+p2_hlen+c_offset+rear_wheels_offset[1]} ${c_offset+p9_len}" />
   </xacro:macro>
 </robot>

File: software/src/pvcchair_description/urdf/includes/parameters.xacro (robot description, xacro)
@@ -1,18 +1,20 @@
 <?xml version="1.0"?>
 <robot name="parameters" xmlns:xacro="http://www.ros.org/wiki/xacro">
-  <xacro:property name="p1_len" value="0.203200" />  <!-- in meters -->
-  <xacro:property name="p2_len" value="0.241300" />
-  <xacro:property name="p3_len" value="0.101600" />
-  <xacro:property name="p4_len" value="0.088900" />
-  <xacro:property name="p5_len" value="0.152400" />
-  <xacro:property name="p6_len" value="0.146050" />
-  <xacro:property name="p7_len" value="0.285750" />
-  <xacro:property name="p8_len" value="0.038100" />
-  <xacro:property name="p9_len" value="0.038100" />
+  <xacro:property name="scale" value="1.2" />
+  <xacro:property name="p1_len" value="${scale*0.203200}" />  <!-- in meters -->
+  <xacro:property name="p2_len" value="${scale*0.241300}" />
+  <xacro:property name="p3_len" value="${scale*0.101600}" />
+  <xacro:property name="p4_len" value="${scale*0.088900}" />
+  <xacro:property name="p5_len" value="${scale*0.152400}" />
+  <xacro:property name="p6_len" value="${scale*0.146050}" />
+  <xacro:property name="p7_len" value="${scale*0.285750}" />
+  <xacro:property name="p8_len" value="${scale*0.038100}" />
+  <xacro:property name="p9_len" value="${scale*0.038100}" />
   <xacro:property name="c_offset" value="0.0127" />
-  <xacro:property name="wheel_radius" value="0.0762" />
+  <xacro:property name="wheel_radius" value="0.07" />
   <xacro:property name="caster_radius" value="0.0508" />
-  <xacro:property name="swivel_offset" value="0.02" />
-  <xacro:property name="base_level" value="0.12" />
+  <xacro:property name="front_wheels_offset" value="${[-0.042, 0.035]}" />
+  <xacro:property name="rear_wheels_offset" value="${[0.02, 0.0]}" />
+  <xacro:property name="base_level" value="0.16" />
   <xacro:property name="back_angle_deg" value="20" />
   <xacro:property name="rest_angle_deg" value="48.8" />
@@ -28,6 +30,6 @@
   <xacro:property name="p8_hlen" value="${p8_len/2}" />
   <xacro:property name="p9_hlen" value="${p9_len/2}" />
-  <xacro:property name="back_angle_rad" value="${back_angle_deg*pi/180}" />
-  <xacro:property name="rest_angle_rad" value="${rest_angle_deg*pi/180}" />
-  <xacro:property name="lock_angle_rad" value="${lock_angle_deg*pi/180}" />
+  <xacro:property name="back_angle_rad" value="${radians(back_angle_deg)}" />
+  <xacro:property name="rest_angle_rad" value="${radians(rest_angle_deg)}" />
+  <xacro:property name="lock_angle_rad" value="${radians(lock_angle_deg)}" />
 </robot>
