Commit message: Remove gearbox plate

File: software/src/pvcchair_description/urdf/includes/components/base.xacro (robot description, xacro)
@@ -24,6 +24,4 @@
       <xacro:p3 xyz="${+p1_hlen+c_offset} ${-p2_hlen-c_offset} ${+p3_hlen+c_offset}" rpy="0 0 0" />
       <xacro:p3 xyz="${+p1_hlen+c_offset} ${+p2_hlen+c_offset} ${+p3_hlen+c_offset}" rpy="0 0 0" />
-      <xacro:p4 xyz="${+p1_hlen+c_offset} ${-p2_hlen-c_offset} ${-p4_hlen-c_offset}" rpy="0 0 0" />
-      <xacro:p4 xyz="${+p1_hlen+c_offset} ${+p2_hlen+c_offset} ${-p4_hlen-c_offset}" rpy="0 0 0" />
       <xacro:p4 xyz="${+p1_hlen+2*c_offset+p4_hlen} ${-p2_hlen-c_offset} 0" rpy="0 ${pi/2} 0" />
       <xacro:p4 xyz="${+p1_hlen+2*c_offset+p4_hlen} ${+p2_hlen+c_offset} 0" rpy="0 ${pi/2} 0" />

File: software/src/pvcchair_description/urdf/includes/components/drive.xacro (robot description, xacro)
@@ -3,23 +3,14 @@
   <xacro:include filename="$(find pvcchair_description)/urdf/includes/parameters.xacro" />
   <xacro:include filename="$(find pvcchair_description)/urdf/includes/parts/caster.xacro" />
-  <xacro:include filename="$(find pvcchair_description)/urdf/includes/parts/gearbox_plate.xacro" />
   <xacro:include filename="$(find pvcchair_description)/urdf/includes/parts/wheel.xacro" />
   <xacro:macro name="drive" params="parent">
-    <xacro:gearbox_plate
+    <xacro:wheel
       suffix="right"
       parent="${parent}"
-      xyz="${p1_hlen+c_offset+gearbox_plate_offset} ${-p2_hlen-c_offset-0.015} ${gearbox_plate_offset}" />
-    <xacro:gearbox_plate
+      xyz="${p1_hlen+c_offset-0.042} ${-p2_hlen-c_offset-0.015-0.02} -0.044" />
+    <xacro:wheel
       suffix="left"
       parent="${parent}"
-      xyz="${p1_hlen+c_offset+gearbox_plate_offset} ${+p2_hlen+c_offset+0.015} ${gearbox_plate_offset}" />
-    <xacro:wheel
-      suffix="right"
-      parent="gearbox_plate_right_link"
-      xyz="-0.052 -0.02 -0.054" />
-    <xacro:wheel
-      suffix="left"
-      parent="gearbox_plate_left_link"
-      xyz="-0.052 +0.02 -0.054" />
+      xyz="${p1_hlen+c_offset-0.042} ${+p2_hlen+c_offset+0.015+0.02} -0.044" />
     <xacro:caster
       suffix="right"

File: software/src/pvcchair_description/urdf/includes/parameters.xacro (robot description, xacro)
@@ -11,5 +11,4 @@
   <xacro:property name="p9_len" value="0.038100" />
   <xacro:property name="c_offset" value="0.0127" />
-  <xacro:property name="gearbox_plate_offset" value="0.01" />
   <xacro:property name="wheel_radius" value="0.0762" />
   <xacro:property name="caster_radius" value="0.0508" />

Commit message: Add swerve wheels

File: software/src/pvcchair_description/urdf/includes/components/base.xacro (robot description, xacro)
@@ -46,4 +46,6 @@
       <xacro:p9 xyz="${-p1_hlen-2*c_offset-p3_len-c_offset} ${-p2_hlen-c_offset} ${+c_offset+p9_len+2*c_offset+p9_hlen}" rpy="0 0 0" />
       <xacro:p9 xyz="${-p1_hlen-2*c_offset-p3_len-c_offset} ${+p2_hlen+c_offset} ${+c_offset+p9_len+2*c_offset+p9_hlen}" rpy="0 0 0" />
+      <xacro:p4 xyz="${-p1_hlen-2*c_offset-p3_len-c_offset} ${-p2_hlen-c_offset} ${+c_offset+p9_len+c_offset-p4_hlen}" rpy="0 0 0" />
+      <xacro:p4 xyz="${-p1_hlen-2*c_offset-p3_len-c_offset} ${+p2_hlen+c_offset} ${+c_offset+p9_len+c_offset-p4_hlen}" rpy="0 0 0" />
     </link>
     <joint name="base_joint" type="fixed">

File: software/src/pvcchair_description/urdf/includes/components/drive.xacro (robot description, xacro)
@@ -2,23 +2,28 @@
 <robot name="motion" xmlns:xacro="http://www.ros.org/wiki/xacro">
   <xacro:include filename="$(find pvcchair_description)/urdf/includes/parameters.xacro" />
-  <xacro:include filename="$(find pvcchair_description)/urdf/includes/parts/caster.xacro" />
-  <xacro:include filename="$(find pvcchair_description)/urdf/includes/parts/wheel.xacro" />
+  <xacro:include filename="$(find pvcchair_description)/urdf/includes/parts/swerve_wheel.xacro" />
   <xacro:macro name="drive" params="parent">
-    <xacro:wheel
-      suffix="right"
+    <xacro:swerve_wheel
+      prefix="fr"
       parent="${parent}"
-      xyz="${p1_hlen+c_offset+front_wheels_offset[0]} ${-p2_hlen-c_offset-front_wheels_offset[1]} ${-base_level+wheel_radius}" />
-    <xacro:wheel
-      suffix="left"
+      x="${p1_hlen+c_offset+front_wheels_offset[0]}"
+      y="${-p2_hlen-c_offset-front_wheels_offset[1]}"
+      yaw="${radians(180)}" />
+    <xacro:swerve_wheel
+      prefix="fl"
       parent="${parent}"
-      xyz="${p1_hlen+c_offset+front_wheels_offset[0]} ${+p2_hlen+c_offset+front_wheels_offset[1]} ${-base_level+wheel_radius}" />
-    <xacro:caster
-      suffix="right"
+      x="${p1_hlen+c_offset+front_wheels_offset[0]}"
+      y="${+p2_hlen+c_offset+front_wheels_offset[1]}" />
+    <xacro:swerve_wheel
+      prefix="br"
       parent="${parent}"
-      xyz="${-p1_hlen-2*c_offset-p3_len-c_offset+rear_wheels_offset[0]} ${-p2_hlen-c_offset-rear_wheels_offset[1]} ${c_offset+p9_len}" />
-    <xacro:caster
-      suffix="left"
+      x="${-p1_hlen-2*c_offset-p3_len-c_offset+rear_wheels_offset[0]}"
+      y="${-p2_hlen-c_offset-front_wheels_offset[1]}"
+      yaw="${radians(180)}" />
+    <xacro:swerve_wheel
+      prefix="bl"
       parent="${parent}"
-      xyz="${-p1_hlen-2*c_offset-p3_len-c_offset+rear_wheels_offset[0]} ${+p2_hlen+c_offset+rear_wheels_offset[1]} ${c_offset+p9_len}" />
+      x="${-p1_hlen-2*c_offset-p3_len-c_offset+rear_wheels_offset[0]}"
+      y="${+p2_hlen+c_offset+front_wheels_offset[1]}" />
   </xacro:macro>
 </robot>

File: software/src/pvcchair_description/urdf/includes/parameters.xacro (robot description, xacro)
@@ -13,8 +13,7 @@
   <xacro:property name="c_offset" value="0.0127" />
   <xacro:property name="wheel_radius" value="0.07" />
-  <xacro:property name="caster_radius" value="0.0508" />
-  <xacro:property name="front_wheels_offset" value="${[-0.042, 0.035]}" />
-  <xacro:property name="rear_wheels_offset" value="${[0.02, 0.0]}" />
-  <xacro:property name="base_level" value="0.16" />
+  <xacro:property name="front_wheels_offset" value="${[0, 0.04]}" />
+  <xacro:property name="rear_wheels_offset" value="${[0, 0.04]}" />
+  <xacro:property name="base_level" value="0.19" />
   <xacro:property name="back_angle_deg" value="20" />
   <xacro:property name="rest_angle_deg" value="48.8" />
